File: KICAD/EGA/EGA.kicad_pcb (KiCad board)
At the start: 2 copper layers, 37 parts, among them J1 12V, J2 HC-SR04, J3 LCD 20x4, J4 RTC, J5 MEMORY SD, J6 FAN_12V_PWM_3.3V, SW1 PAGINA, SW2 RESET, U1 LM7805_TO220, U2 LM317_TO-220, U3 Pico

Commit message: Adicion de PCB_Preliminar para entregar en la segunda parte
Parts:
- removed J5: MEMORY SD, Connector_PinHeader_2.00mm:PinHeader_1x06_P2.00mm_Vertical
- added J7: SD CARD, Connector_PinHeader_2.54mm:PinHeader_1x08_P2.54mm_Vertical, F.Cu at (97.5, 31.4)
- J2, J3, J4, J6: footprint Connector_PinHeader_2.00mm:PinHeader_1x04_P2.00mm_Vertical -> Connector_PinHeader_2.54mm:PinHeader_1x04_P2.54mm_Vertical
- SW1, SW2: footprint Button_Switch_THT:SW_PUSH_6mm_H4.3mm -> Button_Switch_THT:SW_PUSH_6mm_H5mm
- moved H2 190.3 mm to (189.3, 30.6)
- moved R8 158.4 mm to (150.5, 63.0), turned to -90 degrees
- moved H3 154.7 mm to (189.2, 151.9)
- moved RV1 150.9 mm to (155.1, 63.0), turned to -90 degrees
- moved C2 128.0 mm to (147.1, 65.5), turned to -90 degrees
- moved C4 119.7 mm to (124.4, 132.8)
- moved C5 119.2 mm to (136.9, 136.5), turned to 0 degrees
- moved U1 118.6 mm to (110.9, 125.2), turned to -90 degrees
- moved C1 117.9 mm to (98.3, 125.2)
- moved C6 117.9 mm to (103.3, 125.2)
- moved C7 117.9 mm to (93.3, 125.2)
- moved J1 117.9 mm to (85.3, 127.7)
- moved D1 116.6 mm to (119.4, 122.6), turned to -90 degrees
- moved R5 116.0 mm to (99.3, 143.0), turned to 180 degrees
- moved C3 115.8 mm to (103.3, 133.6), turned to 90 degrees
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Connections:
- J6 pad 3: PIN_PRM -> PIN_RPM
- U3 pad 13: unconnected-(U3-GND-Pad13) -> GND
- U3 pad 14: PIN_RPM -> PIN_PWM
- U3 pad 15: PIN_PWM -> PIN_RPM
- U3 pad 18: unconnected-(U3-GND-Pad18) -> GND
- U3 pad 2: PIN_TX -> PIN_TX_MOSI
- U3 pad 23: unconnected-(U3-GND-Pad23) -> GND
- U3 pad 3: GND -> unconnected-(U3-GND-Pad3)
- U3 pad 4: PIN_RX -> PIN_RX_MISO
- U3 pad 8: unconnected-(U3-GND-Pad8) -> GND
Routing:
- net GND: track 171.8 -> 478.5 mm, vias 0 -> 4
- net 5V: track 39.1 -> 284.3 mm, vias 0 -> 2
- net 3.3V: track 32.3 -> 169.6 mm
- net PIN_ADC: track 0.00 -> 57.3 mm
- net PIN_CS: track 0.00 -> 42.3 mm
- net PIN_RPM: track 0.00 -> 34.6 mm
- net PIN_SCK: track 0.00 -> 34.1 mm
- net PIN_PAGINA: track 0.00 -> 33.2 mm
- net VCC: track 33.0 -> 58.3 mm
- net PIN_TX_MOSI: track 0.00 -> 22.4 mm
- net PIN_RX_MISO: track 0.00 -> 22.4 mm
- net Net-(U3-RUN): track 10.9 -> 30.0 mm
- net Net-(D5-A): track 0.00 -> 10.0 mm
- net Net-(SW2-Pad2): track 25.2 -> 15.3 mm
- net Net-(D4-A): track 0.00 -> 9.36 mm
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Other:
- board text added: "BUSTAMANTE PORTAS 5°11 TD3 UTN-FRA"
