File: KICAD/EGA/EGA.kicad_sch (KiCad schematic)
At the start: 39 parts, among them J1 12V, J10 TEST_TRIG, J2 HC-SR04, J3 LCD 20x4, J4 RTC, J5 TEST_PWM, J6 FAN_12V_PWM_3.3V, J7 UART, J8 TEST_RPM, J9 TEST_ECHO, SW1 PAGINA, SW2 RESET, U1 LM7805_TO220, U2 LM317_TO-220, U3 Pico

Commit message: Actualizacion de informe
Parts:
- H1: value MountingHole -> SD
- H2: value MountingHole -> SI
- H3: value MountingHole -> ID
- H4: value MountingHole -> II
Other:
- moved on the sheet: C1, C2, C3, C5, C6, D1, D4, D5, H1, H2, H3, H4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

Commit message: features/Rama Agregado de SD
Parts:
- removed RV1: SetPoint, Potentiometer_THT:Potentiometer_Vishay_T93XA_Horizontal, symbol Device:R_Potentiometer
- added J11: POTENCIOMETRO, Connector_PinHeader_2.54mm:PinHeader_1x03_P2.54mm_Vertical, symbol Connector_Generic:Conn_01x03
- J7: footprint Connector_PinHeader_2.54mm:PinHeader_1x08_P2.54mm_Vertical -> Connector_PinHeader_2.54mm:PinHeader_1x10_P2.54mm_Vertical; symbol Connector_Generic:Conn_01x08 -> Connector_Generic:Conn_01x10
- SW1, SW2: footprint Button_Switch_THT:SW_PUSH_6mm_H5mm -> Button_Switch_THT:SW_PUSH_6mm_H8mm
Connections:
- net 3.3V: now also J11.3 (Pin_3)
- net 5V: now also J7.1 (Pin_1)
- net GND: now also J7.4 (Pin_4), U3.3 (GND), J11.1 (Pin_1); no longer SW2.2, U3.38 (GND)
- net PIN_ADC: now also J11.2 (Pin_2)
- net SCL_1: now also J7.10 (Pin_10); no longer J7.6 (Pin_6)
- net SDA_1: now also J7.9 (Pin_9); no longer J7.5 (Pin_5)
- net UART1_RX: now also J7.8 (Pin_8); no longer J7.4 (Pin_4)
- net UART1_TX: now also J7.7 (Pin_7); no longer J7.3 (Pin_3)
- net SCK/SPI0: now reaches U3.4 (GPIO2)
- net SCK/SPI0: now also J7.5 (Pin_5)
- net TX/SPI0: now reaches U3.5 (GPIO3)
- net TX/SPI0: now also J7.6 (Pin_6)
- net UART0_RX renamed CSn/SPI0
- net CSn/SPI0: now also J7.3 (Pin_3); no longer J7.2 (Pin_2)
- net UART0_TX renamed RX/SPI0
- net RX/SPI0: now also J7.2 (Pin_2); no longer J7.1 (Pin_1)
- new net: SW2.2, U3.38 (GND)
- no-connect marks 26 -> 21
